File: SAMD21 breakout.kicad_sch (KiCad schematic)
At the start: 35 parts, among them J1 USB_B_Micro, J2 Conn_ARM_JTAG_SWD_10, J4 Conn_01x14, J5 Conn_01x18, SW1 SW_Push, U1 ATSAMD21G18A-AU, U2 AMS1117-3.3, Y1 32768Hz

Commit message: Mounting holes do not need be on BOM.
Parts:
- H1, H2, H3, H4: now left out of the parts list
Changed lines of the file:
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@@
   )
   (symbol (lib_id "Mechanical:MountingHole") (at 21.59 182.88 0) (unit 1)
-    (in_bom yes) (on_board yes) (fields_autoplaced)
+    (in_bom no) (on_board yes) (fields_autoplaced)
     (property "Reference" "H3" (id 0) (at 24.13 181.6099 0)
       (effects (font (size 1.27 1.27)) (justify left))
@@
   )
   (symbol (lib_id "Mechanical:MountingHole") (at 21.59 175.26 0) (unit 1)
-    (in_bom yes) (on_board yes) (fields_autoplaced)
+    (in_bom no) (on_board yes) (fields_autoplaced)
     (property "Reference" "H2" (id 0) (at 24.13 173.9899 0)
       (effects (font (size 1.27 1.27)) (justify left))
@@
   )
   (symbol (lib_id "Mechanical:MountingHole") (at 21.59 167.64 0) (unit 1)
-    (in_bom yes) (on_board yes) (fields_autoplaced)
+    (in_bom no) (on_board yes) (fields_autoplaced)
     (property "Reference" "H1" (id 0) (at 24.13 166.3699 0)
       (effects (font (size 1.27 1.27)) (justify left))
@@
   )
   (symbol (lib_id "Mechanical:MountingHole") (at 21.59 190.5 0) (unit 1)
-    (in_bom yes) (on_board yes) (fields_autoplaced)
+    (in_bom no) (on_board yes) (fields_autoplaced)
     (property "Reference" "H4" (id 0) (at 24.13 189.2299 0)
       (effects (font (size 1.27 1.27)) (justify left))
